Commit message: add navigation pkg

File: robot_description/urdf/robot.gazebo.xacro (robot description, xacro)
@@ -11,4 +11,12 @@
       <wheel_separation>${wheel_separation}</wheel_separation>
       <wheel_radius>${wheel_radius}</wheel_radius>
+      <min_linear_velocity>-0.3</min_linear_velocity>
+      <max_linear_velocity>0.6</max_linear_velocity>
+      <min_angular_velocity>-3.6</min_angular_velocity>
+      <max_angular_velocity>3.6</max_angular_velocity>
+      <min_linear_acceleration>-1.5</min_linear_acceleration>
+      <max_linear_acceleration>1.5</max_linear_acceleration>
+      <min_angular_acceleration>-3.0</min_angular_acceleration>
+      <max_angular_acceleration>3.0</max_angular_acceleration>
       <topic>cmd_vel</topic>
       <odom_topic>odom</odom_topic>

File: robot_description/urdf/robot.xacro (robot description, xacro)
@@ -83,5 +83,5 @@
       <origin xyz="${wheel_offset_x} ${reflect * wheel_separation/2} ${wheel_z_offset}" rpy="0 0 0"/>
       <axis xyz="0 1 0"/>
-      <limit effort="50000" velocity="10"/>
+      <limit effort="50000" velocity="30"/>
       <dynamics damping="1.0" friction="1.0"/>
     </joint>
